Commit message: feat: unify M1A MoveIt and Gazebo robot model

File: robot_ws/src/xh_sim/urdf/panda_controlled.urdf (robot description, URDF)
Before this commit: robot xh_panda_controlled, 12 links, 11 joints
Joints:
- joint world_to_panda: origin (none) -> xyz=-0.35 0 0.45 rpy=0 0 0

Commit message: Apply approved Panda kinematics and placement scene

File: robot_ws/src/xh_sim/urdf/panda_controlled.urdf (robot description, URDF)
Before this commit: robot xh_panda_controlled, 12 links, 11 joints
Links:
- added link panda_link8, mass 0.2; collision box size=0.08 0.08 0.08; visual box size=0.08 0.08 0.08
- link panda_link1: geometry collision cylinder length=0.333 radius=0.055; visual cylinder length=0.333 radius=0.055
- link panda_link2: geometry collision box size=0.08 0.316 0.08; visual box size=0.08 0.316 0.08
- link panda_link3: geometry collision box size=0.0825 0.08 0.08; visual box size=0.0825 0.08 0.08
- link panda_link4: geometry collision box size=0.392771 0.08 0.08; visual box size=0.392771 0.08 0.08
- link panda_link5: geometry collision box size=0.10 0.10 0.12; visual box size=0.10 0.10 0.12
- link panda_link6: geometry collision box size=0.088 0.08 0.08; visual box size=0.088 0.08 0.08
- link panda_link7: geometry collision box size=0.08 0.08 0.107; visual box size=0.08 0.08 0.107
Joints:
- added joint panda_joint8: type fixed, parent panda_link7, child panda_link8, origin xyz=0 0 0.107 rpy=0 0 0
- joint panda_hand_joint: origin xyz=0 0 0.18 rpy=0 0 0 -> xyz=0 0 0 rpy=0 0 -0.785398163397; parent panda_link7 -> panda_link8
- joint panda_joint1: origin xyz=0 0 0.16 rpy=0 0 0 -> xyz=0 0 0.333 rpy=0 0 0
- joint panda_joint2: origin xyz=0 0 0.32 rpy=-1.57079632679 0 0 -> xyz=0 0 0 rpy=-1.57079632679 0 0
- joint panda_joint3: origin xyz=0 0 0.32 rpy=1.57079632679 0 0 -> xyz=0 -0.316 0 rpy=1.57079632679 0 0
- joint panda_joint4: origin xyz=0 0 0.30 rpy=1.57079632679 0 0 -> xyz=0.0825 0 0 rpy=1.57079632679 0 0
- joint panda_joint5: origin xyz=0 0 0.26 rpy=-1.57079632679 0 0 -> xyz=-0.0825 0.384 0 rpy=-1.57079632679 0 0
- joint panda_joint6: origin xyz=0 0 0.24 rpy=1.57079632679 0 0 -> xyz=0 0 0 rpy=1.57079632679 0 0
- joint panda_joint7: origin xyz=0 0 0.20 rpy=1.57079632679 0 0 -> xyz=0.088 0 0 rpy=1.57079632679 0 0

Commit message: milestone: verify executed motion, grasp gate, and b1 oracle

File: robot_ws/src/xh_sim/urdf/panda_controlled.urdf (robot description, URDF)
Before this commit: robot xh_panda_controlled, 13 links, 12 joints
Links:
- link panda_link1: geometry collision box size=0.110148 0.184565 0.246977; visual box size=0.110148 0.184565 0.246977
- link panda_link2: geometry collision mesh filename=package://moveit_resources_panda_description/meshes/collisi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; visual box size=0.05 0.316 0.05
- link panda_link3: geometry collision box size=0.0825 0.05 0.05; visual box size=0.0825 0.05 0.05
- link panda_link4: geometry collision mesh filename=package://moveit_resources_panda_description/meshes/collisi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; visual box size=0.192746 0.179159 0.166259
- link panda_link5: geometry collision box size=0.06 0.06 0.08; visual box size=0.06 0.06 0.08
- link panda_link6: geometry collision box size=0.088 0.05 0.05; visual box size=0.088 0.05 0.05
- link panda_link7: geometry collision box size=0.05 0.05 0.08; visual box size=0.05 0.05 0.08
- link panda_link8: geometry collision box size=0.04 0.04 0.04; visual box size=0.04 0.04 0.04
Joints:
- joint panda_finger_joint1: mimic (none) -> joint=panda_finger_joint2 multiplier=1 offset=0

Commit message: feat: apply ADR-0014 grasp geometry revision

File: robot_ws/src/xh_sim/urdf/panda_controlled.urdf (robot description, URDF)
Before this commit: robot xh_panda_controlled, 13 links, 12 joints
Links:
- link panda_hand: geometry collision box size=0.07 0.06 0.11; visual box size=0.07 0.06 0.11
- link panda_leftfinger: geometry collision box size=0.02 0.006 0.012; collision box size=0.08 0.010 0.022
- link panda_rightfinger: geometry collision box size=0.02 0.006 0.012; collision box size=0.08 0.010 0.022

Commit message: feat: adopt ADR0016 inline top grasp topology

File: robot_ws/src/xh_sim/urdf/panda_controlled.urdf (robot description, URDF)
Before this commit: robot xh_panda_controlled, 13 links, 12 joints
Links:
- link panda_hand: geometry collision box size=0.07 0.06 0.06; visual box size=0.07 0.06 0.06
- link panda_leftfinger: geometry collision box size=0.012 0.006 0.02; collision box size=0.022 0.010 0.08
- link panda_rightfinger: geometry collision box size=0.012 0.006 0.02; collision box size=0.022 0.010 0.08
Joints:
- joint panda_finger_joint1: origin xyz=0 0 0.055 rpy=0 0 0 -> xyz=0 0 0.06 rpy=0 0 0
- joint panda_finger_joint2: origin xyz=0 0 0.055 rpy=0 0 0 -> xyz=0 0 0.06 rpy=0 0 0
