Commit message: feat: adopt ADR-0016 §4 franka-copy fallback hand; first nonzero M1B envelope
The ADR-0016 inline hand measured a zero tolerance envelope on every axis
(zero-offset X/Y/Z = 0/3), the pre-authorized §4 trigger. Replace the hand
with a primitive-approximated copy of the official franka_description
geometry (same joint contract) and revalidate.

Diagnosis of the inline 0/9 zero-offset failures (node2 per-trial raws):
three independent mechanisms, none the pad topology — a zero-force kiss-gap
close, an OMPL joint-space descent that bowed and shoved the free target
10-18 mm, and slot-3 pregrasp IK -31 (the §3 scan's target).

Fallback also compensates three measured bullet-featherstone behaviours:
spawned multibody collides only each link's first collision element (grasp
plate moved there); shallow-penetration dead band rejects small convex pads
(grasp element is a full-length plate, face 6.5 mm proud, public gap map
2q-6mm); per-pair force-response lottery cured by a two-stage close. Final
descent is seeded-waypoint straight cartesian; yaw from label free-gap.

Revalidation: bullet audit / home self-collision / S0 13/13 / S1 10/10 pass;
§3 corridor-extended pre-scan admits scene-5017 slots 1/2/4; height/squeeze
frozen at 120 mm / 2 mm / two-stage; 81-trial envelope X 0.015 / Y 0.015 /
Z 0.005 m (summary SHA-256 1e758295...); ADR-0013 acceptance 3 round-trip
passes. Perception p90 gate stays NO_GO but now measured (p90 > 0.6x
envelope, worst on Z), a perception-accuracy problem. Unit suite 110/110.

Follow-ups: perception p90 (near-pregrasp reobservation), ADR-0013
acceptance 4 live wrong-object drill, §3 scan integration into industrial
scene generation, M1A cube regression.

Co-Authored-By: Claude Opus 4.8 (1M context) <noreply@anthropic.com>

File: robot_ws/src/xh_sim/urdf/panda_controlled.urdf (robot description, URDF)
Before this commit: robot xh_panda_controlled, 13 links, 12 joints
Links:
- link panda_hand: geometry collision box size=0.0633 0.2044 0.0919; visual box size=0.0633 0.2044 0.0919
- link panda_leftfinger: geometry collision box size=0.021 0.0208 0.0538; collision box size=0.021 0.0239 0.036
- link panda_rightfinger: geometry collision box size=0.021 0.0208 0.0538; collision box size=0.021 0.0239 0.036
Joints:
- joint panda_finger_joint1: origin xyz=0 0 0.06 rpy=0 0 0 -> xyz=0 0 0.0584 rpy=0 0 0
- joint panda_finger_joint2: origin xyz=0 0 0.06 rpy=0 0 0 -> xyz=0 0 0.0584 rpy=0 0 0
